Commit message: done with description

File: my_robot_description/urdf/common_properties.xacro (robot description, xacro)
@@ -7,5 +7,5 @@
         <color rgba="0.5 0.5 0.5 1.0" />
     </material>
-    <xacro:macro name="box_intertia" params="m x y z o_xyz o_rpy">
+    <xacro:macro name="box_inertia" params="m x y z o_xyz o_rpy">
         <inertial>
             <mass value="${m}" />

File: my_robot_description/urdf/mobile_base.xacro (robot description, xacro)
@@ -21,5 +21,5 @@
             <origin xyz="0 0 ${base_height / 2.0}" rpy="0 0 0" />
         </collision>
-        <xacro:box_intertia m="5.0" x="${base_length}" y="${base_width}" z="${base_height}"
+        <xacro:box_inertia m="5.0" x="${base_length}" y="${base_width}" z="${base_height}"
             o_xyz="0 0 ${base_height / 2.0}" o_rpy="0 0 0" />
     </link>

File: my_robot_description/urdf/my_robot.urdf.xacro (robot description, xacro)
@@ -3,4 +3,5 @@
     <xacro:include filename="common_properties.xacro" />
     <xacro:include filename="mobile_base.xacro" />
-    <xacro:include filename="mobile_base_gazebo.xacro"/>
+    <xacro:include filename="mobile_base_gazebo.xacro" />
+    <xacro:include filename="camera.xacro" />
 </robot>
